File: SchemaElettrico-PCB/Ziliani-Sistema_Irrigazione.brd (EAGLE design)
At the start: 101.6 x 117.8 mm, 10 parts, among them IC1 DS1307, Q1 32768 Hz, U1 ARDUINOR3-DIMENSION

Commit message: Add files via upload
Routing:
- net N$21: track 78.0 -> 112.2 mm
- net N$24: track 13.6 -> 15.1 mm
- net N$25: track 14.3 -> 15.1 mm
- net N$26: track 14.3 -> 13.6 mm
- net N$13: track 233.3 -> 232.8 mm
Changed lines of the file:
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@@
 <wire x1="15.24" y1="74.93" x2="11.43" y2="78.74" width="0.8128" layer="16"/>
 <contactref element="IC1" pad="3"/>
-<wire x1="11.43" y1="78.74" x2="11.43" y2="90.17" width="0.4064" layer="16"/>
+<wire x1="11.43" y1="78.74" x2="11.43" y2="90.17" width="0.8128" layer="16"/>
 </signal>
 <signal name="N$3">
@@
 <wire x1="81.3011" y1="111.7811" x2="81.28" y2="111.76" width="0.8128" layer="1"/>
 <wire x1="43.18" y1="52.07" x2="43.18" y2="58.42" width="0.8128" layer="1"/>
-<wire x1="81.3011" y1="111.7811" x2="81.3011" y2="96.5411" width="0.4064" layer="1"/>
-<wire x1="81.3011" y1="96.5411" x2="44.45" y2="59.69" width="0.4064" layer="1"/>
-<wire x1="44.45" y1="59.69" x2="43.18" y2="58.42" width="0.4064" layer="1"/>
+<wire x1="67.31" y1="82.55" x2="43.18" y2="58.42" width="0.4064" layer="1"/>
+<wire x1="81.3011" y1="111.7811" x2="81.3011" y2="96.5411" width="0.8128" layer="1"/>
+<wire x1="81.3011" y1="96.5411" x2="43.18" y2="58.42" width="0.8128" layer="1"/>
 </signal>
 <signal name="N$13">
@@
 <via x="8.89" y="104.14" extent="1-16" drill="0.9"/>
 <wire x1="8.89" y1="104.14" x2="6.35" y2="101.6" width="0.8128" layer="16"/>
-<wire x1="95.15" y1="97.89" x2="95.15" y2="63.44" width="0.8128" layer="16"/>
-<wire x1="96.42" y1="62.17" x2="95.15" y2="63.44" width="0.8128" layer="16"/>
-<wire x1="95.15" y1="97.89" x2="88.9" y2="104.14" width="0.8128" layer="16"/>
+<wire x1="96.42" y1="96.62" x2="96.42" y2="62.17" width="0.8128" layer="16"/>
+<wire x1="96.42" y1="96.62" x2="88.9" y2="104.14" width="0.8128" layer="16"/>
 <wire x1="88.9" y1="104.14" x2="53.34" y2="104.14" width="0.8128" layer="16"/>
 <wire x1="53.34" y1="104.14" x2="50.8" y2="101.6" width="0.8128" layer="16"/>
@@
 <wire x1="6.35" y1="97.79" x2="5.08" y2="97.79" width="0.8128" layer="16"/>
 <wire x1="50.8" y1="101.6" x2="50.8" y2="100.33" width="0.8128" layer="16"/>
-<wire x1="35.56" y1="43.18" x2="20.32" y2="43.18" width="0.8128" layer="16"/>
-<wire x1="20.32" y1="43.18" x2="15.24" y2="48.26" width="0.8128" layer="16"/>
-<wire x1="7.62" y1="43.18" x2="20.32" y2="43.18" width="0.8128" layer="16"/>
+<wire x1="19.05" y1="43.18" x2="7.62" y2="43.18" width="0.8128" layer="16"/>
+<wire x1="15.24" y1="48.26" x2="15.24" y2="46.99" width="0.8128" layer="16"/>
+<wire x1="15.24" y1="46.99" x2="19.05" y2="43.18" width="0.8128" layer="16"/>
+<wire x1="19.05" y1="43.18" x2="35.56" y2="43.18" width="0.8128" layer="16"/>
 </signal>
 <signal name="N$22">
@@
 <contactref element="U1" pad="D9"/>
 <wire x1="49.784" y1="52.07" x2="47.244" y2="49.53" width="0.4064" layer="16"/>
-<wire x1="47.244" y1="49.53" x2="43.18" y2="49.53" width="0.4064" layer="16"/>
-<wire x1="43.18" y1="49.53" x2="39.37" y2="45.72" width="0.4064" layer="16"/>
-<wire x1="39.37" y1="45.72" x2="39.37" y2="44.45" width="0.4064" layer="16"/>
+<wire x1="47.244" y1="49.53" x2="41.91" y2="49.53" width="0.4064" layer="16"/>
+<wire x1="41.91" y1="49.53" x2="39.37" y2="46.99" width="0.4064" layer="16"/>
+<wire x1="39.37" y1="46.99" x2="39.37" y2="44.45" width="0.4064" layer="16"/>
 </signal>
 <signal name="N$24">
@@
 <contactref element="U1" pad="D10"/>
 <wire x1="48.514" y1="48.26" x2="52.324" y2="52.07" width="0.4064" layer="16"/>
-<wire x1="41.91" y1="44.45" x2="45.72" y2="48.26" width="0.4064" layer="16"/>
-<wire x1="45.72" y1="48.26" x2="48.514" y2="48.26" width="0.4064" layer="16"/>
+<wire x1="43.18" y1="48.26" x2="41.91" y2="46.99" width="0.4064" layer="16"/>
+<wire x1="41.91" y1="44.45" x2="41.91" y2="46.99" width="0.4064" layer="16"/>
+<wire x1="43.18" y1="48.26" x2="48.514" y2="48.26" width="0.4064" layer="16"/>
 </signal>
 <signal name="N$14">
 <contactref element="U1" pad="D11"/>
 <contactref element="U$2" pad="J1.4"/>
-<wire x1="54.864" y1="52.07" x2="54.864" y2="50.8" width="0.4064" layer="16"/>
-<wire x1="54.864" y1="50.8" x2="51.054" y2="46.99" width="0.4064" layer="16"/>
-<wire x1="44.45" y1="44.45" x2="46.99" y2="46.99" width="0.4064" layer="16"/>
-<wire x1="46.99" y1="46.99" x2="51.054" y2="46.99" width="0.4064" layer="16"/>
+<wire x1="54.864" y1="52.07" x2="49.784" y2="46.99" width="0.4064" layer="16"/>
+<wire x1="45.72" y1="46.99" x2="44.45" y2="45.72" width="0.4064" layer="16"/>
+<wire x1="44.45" y1="44.45" x2="44.45" y2="45.72" width="0.4064" layer="16"/>
+<wire x1="45.72" y1="46.99" x2="49.784" y2="46.99" width="0.4064" layer="16"/>
 </signal>
 <signal name="N$26">
@@
 <contactref element="U$2" pad="J1.5"/>
 <wire x1="46.99" y1="44.45" x2="48.26" y2="45.72" width="0.4064" layer="16"/>
-<wire x1="57.404" y1="52.07" x2="57.404" y2="50.8" width="0.4064" layer="16"/>
-<wire x1="57.404" y1="50.8" x2="52.324" y2="45.72" width="0.4064" layer="16"/>
-<wire x1="48.26" y1="45.72" x2="52.324" y2="45.72" width="0.4064" layer="16"/>
+<wire x1="57.404" y1="52.07" x2="51.054" y2="45.72" width="0.4064" layer="16"/>
+<wire x1="48.26" y1="45.72" x2="51.054" y2="45.72" width="0.4064" layer="16"/>
 </signal>
 <signal name="N$8">
